File: lab4/exerciseII.kicad_sch (KiCad schematic)
At the start: 0 parts

Commit message: Updated exerciseII file and added exercise2.txt(annotations)
Parts:
- added C1: 10uF, symbol Device:C_Polarized
- added C2: 0.01uF, symbol Device:C
- added D1, D2: LED, symbol Device:LED
- added J1: (no value), symbol Connector:Conn_01x02_Male
- added R1, R2, R3, R4: 1k, symbol Device:R
- added U1: (no value), Package_SO:SOIC-8_3.9x4.9mm_P1.27mm, symbol Timer:NE555D
Connections:
- new net: D1.1 (K), R2.1
- new net: C2.1, U1.5 (CV)
- new net: D2.2 (A), R4.2
- new net +9V: D1.2 (A), J1.1 (Pin_1), R1.1, U1.4 (R), U1.8 (VCC)
- new net GND: C1.2, C2.2, D2.1 (K), J1.2 (Pin_2), U1.1 (GND)
- new net Pin_2: C1.1, R3.2, U1.2 (TR), U1.6 (THR)
- new net Pin_3: R2.2, R4.1, U1.3 (Q)
- new net Pin_7: R1.2, R3.1, U1.7 (DIS)
Other:
- title: (none) -> 555 Timer Circuit

Commit message: finished PCB layouts
Parts:
- C1: footprint (none) -> Capacitor_Tantalum_SMD:CP_EIA-3216-18_Kemet-A_Pad1.58x1.35mm_HandSolder
- C2: footprint (none) -> Capacitor_SMD:C_0805_2012Metric_Pad1.18x1.45mm_HandSolder
- D1, D2: footprint (none) -> LED_SMD:LED_1206_3216Metric_Pad1.42x1.75mm_HandSolder
- J1: footprint (none) -> TerminalBlock:TerminalBlock_bornier-2_P5.08mm
- R1, R2, R3, R4: footprint (none) -> Resistor_SMD:R_0805_2012Metric_Pad1.20x1.40mm_HandSolder
Changed lines of the file:
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@@
       (effects (font (size 1.27 1.27)) (justify right))
     )
-    (property "Footprint" "" (id 2) (at 135.89 36.83 0)
+    (property "Footprint" "LED_SMD:LED_1206_3216Metric_Pad1.42x1.75mm_HandSolder" (id 2) (at 135.89 36.83 0)
       (effects (font (size 1.27 1.27)) hide)
     )
@@
       (effects (font (size 1.27 1.27)) (justify left))
     )
-    (property "Footprint" "" (id 2) (at 134.112 59.69 90)
+    (property "Footprint" "Resistor_SMD:R_0805_2012Metric_Pad1.20x1.40mm_HandSolder" (id 2) (at 134.112 59.69 90)
       (effects (font (size 1.27 1.27)) hide)
     )
@@
       (effects (font (size 1.27 1.27)) (justify left))
     )
-    (property "Footprint" "" (id 2) (at 134.112 46.99 90)
+    (property "Footprint" "Resistor_SMD:R_0805_2012Metric_Pad1.20x1.40mm_HandSolder" (id 2) (at 134.112 46.99 90)
       (effects (font (size 1.27 1.27)) hide)
     )
@@
       (effects (font (size 1.27 1.27)) (justify left))
     )
-    (property "Footprint" "" (id 2) (at 79.7052 72.39 0)
+    (property "Footprint" "Capacitor_SMD:C_0805_2012Metric_Pad1.18x1.45mm_HandSolder" (id 2) (at 79.7052 72.39 0)
       (effects (font (size 1.27 1.27)) hide)
     )
@@
       (effects (font (size 1.27 1.27)) (justify left))
     )
-    (property "Footprint" "" (id 2) (at 61.9252 72.39 0)
+    (property "Footprint" "Capacitor_Tantalum_SMD:CP_EIA-3216-18_Kemet-A_Pad1.58x1.35mm_HandSolder" (id 2) (at 61.9252 72.39 0)
       (effects (font (size 1.27 1.27)) hide)
     )
@@
       (effects (font (size 1.27 1.27)) (justify right))
     )
-    (property "Footprint" "" (id 2) (at 135.89 69.85 0)
+    (property "Footprint" "LED_SMD:LED_1206_3216Metric_Pad1.42x1.75mm_HandSolder" (id 2) (at 135.89 69.85 0)
       (effects (font (size 1.27 1.27)) hide)
     )
@@
       (effects (font (size 1.27 1.27)) (justify left))
     )
-    (property "Footprint" "" (id 2) (at 59.182 43.18 90)
+    (property "Footprint" "Resistor_SMD:R_0805_2012Metric_Pad1.20x1.40mm_HandSolder" (id 2) (at 59.182 43.18 90)
       (effects (font (size 1.27 1.27)) hide)
     )
@@
       (effects (font (size 1.27 1.27)) (justify right))
     )
-    (property "Footprint" "" (id 2) (at 73.66 35.56 0)
+    (property "Footprint" "TerminalBlock:TerminalBlock_bornier-2_P5.08mm" (id 2) (at 73.66 35.56 0)
       (effects (font (size 1.27 1.27)) hide)
     )
@@
       (effects (font (size 1.27 1.27)) (justify left))
     )
-    (property "Footprint" "" (id 2) (at 59.182 55.88 90)
+    (property "Footprint" "Resistor_SMD:R_0805_2012Metric_Pad1.20x1.40mm_HandSolder" (id 2) (at 59.182 55.88 90)
       (effects (font (size 1.27 1.27)) hide)
     )
@@
     )
     (path "/93236a74-ceb1-4bd7-9e0e-417e53923d8c"
-      (reference "C1") (unit 1) (value "10uF") (footprint "")
+      (reference "C1") (unit 1) (value "10uF") (footprint "Capacitor_Tantalum_SMD:CP_EIA-3216-18_Kemet-A_Pad1.58x1.35mm_HandSolder")
     )
     (path "/83b90431-2aca-43b3-b964-e864bcbb0ff9"
-      (reference "C2") (unit 1) (value "0.01uF") (footprint "")
+      (reference "C2") (unit 1) (value "0.01uF") (footprint "Capacitor_SMD:C_0805_2012Metric_Pad1.18x1.45mm_HandSolder")
     )
     (path "/00dbe83f-1ca1-4afd-b158-94efc192baae"
-      (reference "D1") (unit 1) (value "LED") (footprint "")
+      (reference "D1") (unit 1) (value "LED") (footprint "LED_SMD:LED_1206_3216Metric_Pad1.42x1.75mm_HandSolder")
     )
     (path "/95a7ec6b-934d-4ae3-b530-bb4676122264"
-      (reference "D2") (unit 1) (value "LED") (footprint "")
+      (reference "D2") (unit 1) (value "LED") (footprint "LED_SMD:LED_1206_3216Metric_Pad1.42x1.75mm_HandSolder")
     )
     (path "/be25aa55-009d-40be-8928-b3f0e353dbef"
-      (reference "J1") (unit 1) (value " ") (footprint "")
+      (reference "J1") (unit 1) (value " ") (footprint "TerminalBlock:TerminalBlock_bornier-2_P5.08mm")
     )
     (path "/a753a813-b813-4838-a41b-43c50606d98c"
-      (reference "R1") (unit 1) (value "1k") (footprint "")
+      (reference "R1") (unit 1) (value "1k") (footprint "Resistor_SMD:R_0805_2012Metric_Pad1.20x1.40mm_HandSolder")
     )
     (path "/48e6bab2-79db-4348-9558-d264ae5e5836"
-      (reference "R2") (unit 1) (value "1k") (footprint "")
+      (reference "R2") (unit 1) (value "1k") (footprint "Resistor_SMD:R_0805_2012Metric_Pad1.20x1.40mm_HandSolder")
     )
     (path "/ef463d7c-60bc-48a0-bfad-714d943573f4"
-      (reference "R3") (unit 1) (value "1k") (footprint "")
+      (reference "R3") (unit 1) (value "1k") (footprint "Resistor_SMD:R_0805_2012Metric_Pad1.20x1.40mm_HandSolder")
     )
     (path "/2b9c8678-c314-43be-9c70-19357cd0d76f"
-      (reference "R4") (unit 1) (value "1k") (footprint "")
+      (reference "R4") (unit 1) (value "1k") (footprint "Resistor_SMD:R_0805_2012Metric_Pad1.20x1.40mm_HandSolder")
     )
     (path "/2518d884-5a2b-4be0-bfb9-fc9bf3e52505"
