File: lab4/exerciseII.kicad_pcb (KiCad board)
At the start: 2 copper layers, 10 parts, among them J1 , U1 

Commit message: added gerber files
Routing:
- net +9V: track 63.3 -> 62.1 mm
Changed lines of the file:
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@@
       (viasonmask false)
       (mode 1)
-      (useauxorigin false)
+      (useauxorigin true)
       (hpglpennumber 1)
       (hpglpenspeed 20)
@@
       (outputformat 1)
       (mirror false)
-      (drillshape 1)
+      (drillshape 0)
       (scaleselection 1)
-      (outputdirectory "")
+      (outputdirectory "./")
     )
   )
@@
     (fp_line (start -1.6 0.8) (end 1.6 0.8) (layer "F.Fab") (width 0.1))
     (fp_line (start -1.2 -0.8) (end -1.6 -0.4) (layer "F.Fab") (width 0.1))
-    (pad "1" smd roundrect (at -1.4875 0) (size 1.425 1.75) (layers "F.Cu" "F.Paste" "F.Mask") (roundrect_rratio 0.175439)
+    (pad "1" smd roundrect (at -1.4875 0) (size 1.425 1.75) (layers "F.Cu" "F.Paste" "F.Mask") (roundrect_rratio 0.1754392982)
       (net 2 "GND") (pinfunction "K") (pintype "passive"))
-    (pad "2" smd roundrect (at 1.4875 0) (size 1.425 1.75) (layers "F.Cu" "F.Paste" "F.Mask") (roundrect_rratio 0.175439)
+    (pad "2" smd roundrect (at 1.4875 0) (size 1.425 1.75) (layers "F.Cu" "F.Paste" "F.Mask") (roundrect_rratio 0.1754392982)
       (net 6 "Net-(D2-Pad2)") (pinfunction "A") (pintype "passive"))
     (model "${KICAD6_3DMODEL_DIR}/LED_SMD.3dshapes/LED_1206_3216Metric.wrl"
@@
     (fp_line (start 1 0.625) (end -1 0.625) (layer "F.Fab") (width 0.1))
     (fp_line (start -1 -0.625) (end 1 -0.625) (layer "F.Fab") (width 0.1))
-    (pad "1" smd roundrect (at -1 0) (size 1.2 1.4) (layers "F.Cu" "F.Paste" "F.Mask") (roundrect_rratio 0.208333)
+    (pad "1" smd roundrect (at -1 0) (size 1.2 1.4) (layers "F.Cu" "F.Paste" "F.Mask") (roundrect_rratio 0.2083333333)
       (net 5 "+9V") (pintype "passive"))
-    (pad "2" smd roundrect (at 1 0) (size 1.2 1.4) (layers "F.Cu" "F.Paste" "F.Mask") (roundrect_rratio 0.208333)
+    (pad "2" smd roundrect (at 1 0) (size 1.2 1.4) (layers "F.Cu" "F.Paste" "F.Mask") (roundrect_rratio 0.2083333333)
       (net 7 "/Pin_7") (pintype "passive"))
     (model "${KICAD6_3DMODEL_DIR}/Resistor_SMD.3dshapes/R_0805_2012Metric.wrl"
@@
     (fp_line (start 1 0.625) (end -1 0.625) (layer "F.Fab") (width 0.1))
     (fp_line (start -1 0.625) (end -1 -0.625) (layer "F.Fab") (width 0.1))
-    (pad "1" smd roundrect (at -1 0 180) (size 1.2 1.4) (layers "F.Cu" "F.Paste" "F.Mask") (roundrect_rratio 0.208333)
+    (pad "1" smd roundrect (at -1 0 180) (size 1.2 1.4) (layers "F.Cu" "F.Paste" "F.Mask") (roundrect_rratio 0.2083333333)
       (net 7 "/Pin_7") (pintype "passive"))
-    (pad "2" smd roundrect (at 1 0 180) (size 1.2 1.4) (layers "F.Cu" "F.Paste" "F.Mask") (roundrect_rratio 0.208333)
+    (pad "2" smd roundrect (at 1 0 180) (size 1.2 1.4) (layers "F.Cu" "F.Paste" "F.Mask") (roundrect_rratio 0.2083333333)
       (net 1 "/Pin_2") (pintype "passive"))
     (model "${KICAD6_3DMODEL_DIR}/Resistor_SMD.3dshapes/R_0805_2012Metric.wrl"
@@
     (fp_line (start 1 0.625) (end -1 0.625) (layer "F.Fab") (width 0.1))
     (fp_line (start 1 -0.625) (end 1 0.625) (layer "F.Fab") (width 0.1))
-    (pad "1" smd roundrect (at -1 0 180) (size 1.2 1.4) (layers "F.Cu" "F.Paste" "F.Mask") (roundrect_rratio 0.208333)
+    (pad "1" smd roundrect (at -1 0 180) (size 1.2 1.4) (layers "F.Cu" "F.Paste" "F.Mask") (roundrect_rratio 0.2083333333)
       (net 8 "/Pin_3") (pintype "passive"))
-    (pad "2" smd roundrect (at 1 0 180) (size 1.2 1.4) (layers "F.Cu" "F.Paste" "F.Mask") (roundrect_rratio 0.208333)
+    (pad "2" smd roundrect (at 1 0 180) (size 1.2 1.4) (layers "F.Cu" "F.Paste" "F.Mask") (roundrect_rratio 0.2083333333)
       (net 6 "Net-(D2-Pad2)") (pintype "passive"))
     (model "${KICAD6_3DMODEL_DIR}/Resistor_SMD.3dshapes/R_0805_2012Metric.wrl"
@@
     (fp_line (start -1 0.625) (end -1 -0.625) (layer "F.Fab") (width 0.1))
     (fp_line (start -1 -0.625) (end 1 -0.625) (layer "F.Fab") (width 0.1))
-    (pad "1" smd roundrect (at -1 0) (size 1.2 1.4) (layers "F.Cu" "F.Paste" "F.Mask") (roundrect_rratio 0.208333)
+    (pad "1" smd roundrect (at -1 0) (size 1.2 1.4) (layers "F.Cu" "F.Paste" "F.Mask") (roundrect_rratio 0.2083333333)
       (net 4 "Net-(D1-Pad1)") (pintype "passive"))
-    (pad "2" smd roundrect (at 1 0) (size 1.2 1.4) (layers "F.Cu" "F.Paste" "F.Mask") (roundrect_rratio 0.208333)
+    (pad "2" smd roundrect (at 1 0) (size 1.2 1.4) (layers "F.Cu" "F.Paste" "F.Mask") (roundrect_rratio 0.2083333333)
       (net 8 "/Pin_3") (pintype "passive"))
     (model "${KICAD6_3DMODEL_DIR}/Resistor_SMD.3dshapes/R_0805_2012Metric.wrl"
@@
     (fp_line (start -1 -0.625) (end 1 -0.625) (layer "F.Fab") (width 0.1))
     (fp_line (start 1 0.625) (end -1 0.625) (layer "F.Fab") (width 0.1))
-    (pad "1" smd roundrect (at -1.0375 0 180) (size 1.175 1.45) (layers "F.Cu" "F.Paste" "F.Mask") (roundrect_rratio 0.212766)
+    (pad "1" smd roundrect (at -1.0375 0 180) (size 1.175 1.45) (layers "F.Cu" "F.Paste" "F.Mask") (roundrect_rratio 0.2127659574)
       (net 3 "Net-(C2-Pad1)") (pintype "passive"))
-    (pad "2" smd roundrect (at 1.0375 0 180) (size 1.175 1.45) (layers "F.Cu" "F.Paste" "F.Mask") (roundrect_rratio 0.212766)
+    (pad "2" smd roundrect (at 1.0375 0 180) (size 1.175 1.45) (layers "F.Cu" "F.Paste" "F.Mask") (roundrect_rratio 0.2127659574)
       (net 2 "GND") (pintype "passive"))
     (model "${KICAD6_3DMODEL_DIR}/Capacitor_SMD.3dshapes/C_0805_2012Metric.wrl"
@@
     (fp_line (start 1.6 -0.8) (end -1.2 -0.8) (layer "F.Fab") (width 0.1))
     (fp_line (start -1.6 -0.4) (end -1.6 0.8) (layer "F.Fab") (width 0.1))
-    (pad "1" smd roundrect (at -1.4875 0) (size 1.425 1.75) (layers "F.Cu" "F.Paste" "F.Mask") (roundrect_rratio 0.175439)
+    (pad "1" smd roundrect (at -1.4875 0) (size 1.425 1.75) (layers "F.Cu" "F.Paste" "F.Mask") (roundrect_rratio 0.1754392982)
       (net 4 "Net-(D1-Pad1)") (pinfunction "K") (pintype "passive"))
-    (pad "2" smd roundrect (at 1.4875 0) (size 1.425 1.75) (layers "F.Cu" "F.Paste" "F.Mask") (roundrect_rratio 0.175439)
+    (pad "2" smd roundrect (at 1.4875 0) (size 1.425 1.75) (layers "F.Cu" "F.Paste" "F.Mask") (roundrect_rratio 0.1754392982)
       (net 5 "+9V") (pinfunction "A") (pintype "passive"))
     (model "${KICAD6_3DMODEL_DIR}/LED_SMD.3dshapes/LED_1206_3216Metric.wrl"
@@
     (fp_line (start 1.6 -0.8) (end -1.2 -0.8) (layer "F.Fab") (width 0.1))
     (fp_line (start -1.6 0.8) (end 1.6 0.8) (layer "F.Fab") (width 0.1))
-    (pad "1" smd roundrect (at -1.4375 0) (size 1.575 1.35) (layers "F.Cu" "F.Paste" "F.Mask") (roundrect_rratio 0.185185)
+    (pad "1" smd roundrect (at -1.4375 0) (size 1.575 1.35) (layers "F.Cu" "F.Paste" "F.Mask") (roundrect_rratio 0.1851851852)
       (net 1 "/Pin_2") (pintype "passive"))
-    (pad "2" smd roundrect (at 1.4375 0) (size 1.575 1.35) (layers "F.Cu" "F.Paste" "F.Mask") (roundrect_rratio 0.185185)
+    (pad "2" smd roundrect (at 1.4375 0) (size 1.575 1.35) (layers "F.Cu" "F.Paste" "F.Mask") (roundrect_rratio 0.1851851852)
       (net 2 "GND") (pintype "passive"))
     (model "${KICAD6_3DMODEL_DIR}/Capacitor_Tantalum_SMD.3dshapes/CP_EIA-3216-18_Kemet-A.wrl"
@@
   (segment (start 26.8375 30.48) (end 29.7025 30.48) (width 0.25) (layer "F.Cu") (net 2))
   (segment (start 22.85 31.143173) (end 23.186827 31.48) (width 0.25) (layer "F.Cu") (net 2))
-  (segment (start 29.8425 30.48) (end 29.7725 30.41) (width 0.25) (layer "F.Cu") (net 2))
   (segment (start 39.45 26.14) (end 39.45 29.29) (width 0.25) (layer "F.Cu") (net 3))
   (segment (start 40.64 40.64) (end 31.8475 31.8475) (width 0.25) (layer "F.Cu") (net 3))
@@
   (segment (start 28.48 33.53) (end 28.48 33.56) (width 0.25) (layer "F.Cu") (net 5))
   (segment (start 40.64 21.14) (end 40.605 21.175) (width 0.25) (layer "F.Cu") (net 5))
-  (segment (start 28.48 33.53) (end 28.45 33.53) (width 0.25) (layer "F.Cu") (net 5))
   (segment (start 40.64 15.24) (end 40.64 21.14) (width 0.25) (layer "F.Cu") (net 5))
   (segment (start 35.655 25.2425) (end 38.4125 28) (width 0.25) (layer "F.Cu") (net 5))
-  (segment (start 39.841751 21.175) (end 40.605 21.175) (width 0.25) (layer "F.Cu") (net 5))
-  (segment (start 35.655 24.985) (end 36.031751 24.985) (width 0.25) (layer "F.Cu") (net 5))
   (segment (start 35.655 24.985) (end 35.655 25.2425) (width 0.25) (layer "F.Cu") (net 5))
   (via (at 30.48 35.56) (size 0.8) (drill 0.4) (layers "F.Cu" "B.Cu") (net 5))
