File: lab4/exercise1/exercise1.kicad_sch (KiCad schematic)
At the start: 6 parts, among them SW1 SW_SPDT

Commit message: finished PCB layouts
Parts:
- C1: footprint (none) -> Capacitor_THT:C_Radial_D5.0mm_H5.0mm_P2.00mm
- D1: footprint (none) -> LED_THT:LED_D5.0mm
- R1, R2: footprint (none) -> Resistor_THT:R_Axial_DIN0516_L15.5mm_D5.0mm_P20.32mm_Horizontal
- SW1: footprint (none) -> Button_Switch_THT:SW_E-Switch_EG1224_SPDT_Angled
- V1: footprint (none) -> Connector_JST:JST_PH_B2B-PH-K_1x02_P2.00mm_Vertical
Changed lines of the file:
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@@
       (effects (font (size 1.27 1.27)) (justify right))
     )
-    (property "Footprint" "" (id 2) (at 71.12 38.1 0)
+    (property "Footprint" "LED_THT:LED_D5.0mm" (id 2) (at 71.12 38.1 0)
       (effects (font (size 1.27 1.27)) hide)
     )
@@
       (effects (font (size 1.27 1.27)) (justify left))
     )
-    (property "Footprint" "" (id 2) (at 69.342 27.94 90)
+    (property "Footprint" "Resistor_THT:R_Axial_DIN0516_L15.5mm_D5.0mm_P20.32mm_Horizontal" (id 2) (at 69.342 27.94 90)
       (effects (font (size 1.27 1.27)) hide)
     )
@@
     (property "Reference" "R2" (id 0) (at 33.02 15.24 90))
     (property "Value" "2.2k" (id 1) (at 33.02 17.78 90))
-    (property "Footprint" "" (id 2) (at 33.02 23.368 90)
+    (property "Footprint" "Resistor_THT:R_Axial_DIN0516_L15.5mm_D5.0mm_P20.32mm_Horizontal" (id 2) (at 33.02 23.368 90)
       (effects (font (size 1.27 1.27)) hide)
     )
@@
       (effects (font (size 1.27 1.27)) (justify left))
     )
-    (property "Footprint" "" (id 2) (at 55.5752 38.1 0)
+    (property "Footprint" "Capacitor_THT:C_Radial_D5.0mm_H5.0mm_P2.00mm" (id 2) (at 55.5752 38.1 0)
       (effects (font (size 1.27 1.27)) hide)
     )
@@
     (property "Reference" "V1" (id 0) (at 24.765 25.4 0))
     (property "Value" "9 V" (id 1) (at 24.765 27.94 0))
-    (property "Footprint" "" (id 2) (at 24.13 30.48 0)
+    (property "Footprint" "Connector_JST:JST_PH_B2B-PH-K_1x02_P2.00mm_Vertical" (id 2) (at 24.13 30.48 0)
       (effects (font (size 1.27 1.27)) hide)
     )
@@
     (property "Reference" "SW1" (id 0) (at 44.45 13.97 0))
     (property "Value" "SW_SPDT" (id 1) (at 44.45 16.51 0))
-    (property "Footprint" "" (id 2) (at 44.45 21.59 0)
+    (property "Footprint" "Button_Switch_THT:SW_E-Switch_EG1224_SPDT_Angled" (id 2) (at 44.45 21.59 0)
       (effects (font (size 1.27 1.27)) hide)
     )
@@
   (symbol_instances
     (path "/8242d33f-c7ca-45a4-9eb9-858bf1a79005"
-      (reference "C1") (unit 1) (value "4.7 MicroF") (footprint "")
+      (reference "C1") (unit 1) (value "4.7 MicroF") (footprint "Capacitor_THT:C_Radial_D5.0mm_H5.0mm_P2.00mm")
     )
     (path "/2a87b80d-4384-4783-8e28-ff023ba56819"
-      (reference "D1") (unit 1) (value "LED") (footprint "")
+      (reference "D1") (unit 1) (value "LED") (footprint "LED_THT:LED_D5.0mm")
     )
     (path "/351ccd2d-dc4e-4c53-8c92-4c076f9cebfd"
-      (reference "R1") (unit 1) (value "20k") (footprint "")
+      (reference "R1") (unit 1) (value "20k") (footprint "Resistor_THT:R_Axial_DIN0516_L15.5mm_D5.0mm_P20.32mm_Horizontal")
     )
     (path "/488d84ac-f605-4b6f-a73e-f1aa40a83fc2"
-      (reference "R2") (unit 1) (value "2.2k") (footprint "")
+      (reference "R2") (unit 1) (value "2.2k") (footprint "Resistor_THT:R_Axial_DIN0516_L15.5mm_D5.0mm_P20.32mm_Horizontal")
     )
     (path "/d6607ed8-b767-410c-8ada-4238712e3032"
-      (reference "SW1") (unit 1) (value "SW_SPDT") (footprint "")
+      (reference "SW1") (unit 1) (value "SW_SPDT") (footprint "Button_Switch_THT:SW_E-Switch_EG1224_SPDT_Angled")
     )
     (path "/cb354bfb-dfc9-4ab0-bab7-72fdeb096213"
-      (reference "V1") (unit 1) (value "9 V") (footprint "")
+      (reference "V1") (unit 1) (value "9 V") (footprint "Connector_JST:JST_PH_B2B-PH-K_1x02_P2.00mm_Vertical")
     )
   )
